Commit message: re-implement-local-planning

File: src/main_bot/description/lidar.xacro (robot description, xacro)
@@ -30,11 +30,7 @@
     <gazebo reference="lidar_frame">
         <sensor name="lidar" type="gpu_lidar">
-            <!-- gz_frame_id stays unprefixed: robot_state_publisher isn't renaming
-                 URDF link names, it just gets its own /<robot_name>/tf topic via
-                 node namespacing, so "lidar_frame" is still the frame it publishes
-                 there. Only the gz-transport topic needs a unique name per robot. -->
             <gz_frame_id>lidar_frame</gz_frame_id>
             <pose>0 0 0 0 0 0</pose>
-            <topic>${frame_prefix}scan</topic>
+            <topic>scan</topic>
             <update_rate>10</update_rate>
             <always_on>1</always_on>

File: src/main_bot/description/robot.urdf.xacro (robot description, xacro)
@@ -1,28 +1,6 @@
 <?xml version="1.0"?>
 <robot xmlns:xacro="http://www.ros.org/wiki/xacro"  name="robot">
-    <!-- Multi-robot support: empty by default so single-robot launches
-         (gz.launch.py, slam.launch.py, nav2.launch.py) are unaffected.
-         Pass robot_name (no slash, e.g. "robot1") to get a ROS namespace
-         for the controller_manager and a "robot1/" tf/topic prefix. -->
-    <xacro:arg name="robot_name" default=""/>
-    <xacro:property name="robot_name" value="$(arg robot_name)"/>
-    <xacro:property name="frame_prefix" value="${'' if robot_name == '' else robot_name + '/'}"/>
-    <!-- ros2_control (via gz_ros2_control) is the default: it's what gz.launch.py /
-         slam.launch.py / nav2.launch.py are built and tested against for a single
-         robot. gz_ros2_control has proven unreliable running multiple controller_manager
-         instances in one Gazebo process, so multi_robot.launch.py sets this false to
-         get the plain gz-sim DiffDrive plugin instead (no per-robot controller_manager). -->
-    <xacro:arg name="use_ros2_control" default="true"/>
-    <xacro:property name="use_ros2_control" value="$(arg use_ros2_control)"/>
-    <!-- Robot_frames -->
     <xacro:include filename = "robot_main.xacro" />
-    <!-- Controls -->
-    <xacro:if value="${use_ros2_control}">
-        <xacro:include filename = "ros2_controller.xacro" />
-    </xacro:if>
-    <xacro:unless value="${use_ros2_control}">
-        <xacro:include filename = "gz_diff_drive.xacro" />
-    </xacro:unless>
-    <!-- Sensors -->
+    <xacro:include filename = "ros2_controller.xacro" />
     <xacro:include filename = "lidar.xacro" />
 </robot>

File: src/main_bot/description/robot_main.xacro (robot description, xacro)
@@ -18,5 +18,4 @@
     <xacro:property name="caster_wheel_offset_front" value="${chassis_length - caster_wheel_radius - caster_wheel_margin}"/>
     <xacro:property name="caster_wheel_offset_rear"  value="${caster_wheel_radius + caster_wheel_margin}"/>
-    <!-- Colors -->
     <material name="white">
         <color rgba= "1 1 1 1"/>
@@ -37,9 +36,6 @@
         <color rgba= "0 0 1 1"/>
     </material>
-    <!-- convention (except base_link): joint followed by link -->
-    <!-- base_link -->
     <link name="base_link">
     </link>
-    <!-- base_footprint -->
     <joint name="base_footprint_joint" type="fixed">
         <parent link= "base_link"/>
@@ -49,5 +45,4 @@
     <link name="base_footprint">
     </link>
-    <!-- chasis -->
     <joint name="chasis_joint" type="fixed">
         <parent link= "base_link"/>
@@ -79,5 +74,4 @@
         </material>
     </gazebo>
-    <!-- left_wheel -->
     <joint name="left_wheel_joint" type="continuous">
         <parent link= "base_link"/>
@@ -108,5 +102,4 @@
         </material>
     </gazebo>
-    <!-- right_wheel -->
     <joint name="right_wheel_joint" type="continuous">
         <parent link= "base_link"/>
@@ -137,5 +130,4 @@
         </material>
     </gazebo>
-    <!-- caster_wheel_front -->
     <joint name="caster_wheel_front_joint" type="fixed">
         <parent link= "chasis"/>
@@ -167,5 +159,4 @@
         <mu2 value= "0.0001"/>
     </gazebo>
-    <!-- caster_wheel_rear -->
     <joint name="caster_wheel_rear_joint" type="fixed">
         <parent link= "chasis"/>

File: src/main_bot/description/ros2_controller.xacro (robot description, xacro)
@@ -26,7 +26,4 @@
                 name="gz_ros2_control::GazeboSimROS2ControlPlugin">
             <parameters>$(find main_bot)/config/controllers.yaml</parameters>
-            <ros>
-                <namespace>${robot_name}</namespace>
-            </ros>
         </plugin>
     </gazebo>
